Commit message: Upload ROS2 project (hyo version)

File: src/my_robot/urdf/turtlebot3_with_sensors.urdf (robot description, URDF)
Before this commit: robot turtlebot3_waffle, 10 links, 9 joints
Links:
- removed link camera_left_link
- removed link camera_right_link
- added link depth_camera_link, mass 0.1; collision box size=0.025 0.09 0.025; visual box size=0.025 0.09 0.025
- link base_link: mass 1.0 -> 1.5
- link velodyne_link: mass 0.83 -> 0.5
Joints:
- removed joint camera_left_joint
- removed joint camera_right_joint
- added joint depth_camera_joint: type fixed, parent base_link, child depth_camera_link, origin xyz=0.073 0 0.084 rpy=0 0 1.5708
- joint velodyne_joint: origin xyz=0 0 0.18 rpy=0 0 0 -> xyz=0 0 0.12 rpy=0 0 0

Commit message: Initial commit: 고인돌 순찰 로봇 Phase 1, 2 완료
- Phase 1: 수동 탐색 및 waypoint 저장
- Phase 2: 자동 순찰
- YOLOv8 object detection
- Navigation2 파라미터 최적화
- 2배 스케일 로봇 URDF

File: src/my_robot/urdf/turtlebot3_with_sensors.urdf (robot description, URDF)
Before this commit: robot turtlebot3_waffle, 9 links, 8 joints
Links:
- link base_link: mass 1.5 -> 6.0; geometry collision box size=0.532 0.532 0.188; visual mesh filename=package://turtlebot3_description/meshes/bases/waffle_base.s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 scale=0.002 0.002 0.002
- link base_scan: mass 0.114 -> 0.456; geometry visual cylinder length=0.063 radius=0.11
- link caster_back_left_link: mass 0.01 -> 0.04
- link caster_back_right_link: mass 0.01 -> 0.04
- link depth_camera_link: mass 0.1 -> 0.4; geometry visual box size=0.05 0.18 0.05
- link velodyne_link: mass 0.5 -> 2.0; geometry visual cylinder length=0.14 radius=0.10
- link wheel_left_link: mass 0.1 -> 0.4; geometry collision cylinder length=0.036 radius=0.066; visual mesh filename=package://turtlebot3_description/meshes/wheels/left_tire.stl scale=0.002 0.002 0.002
- link wheel_right_link: mass 0.1 -> 0.4; geometry collision cylinder length=0.036 radius=0.066; visual mesh filename=package://turtlebot3_description/meshes/wheels/right_tire.s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 scale=0.002 0.002 0.002
Joints:
- joint base_joint: origin xyz=0 0 0.010 rpy=0 0 0 -> xyz=0 0 0.020 rpy=0 0 0
- joint caster_back_left_joint: origin xyz=-0.177 0.064 -0.004 rpy=-1.57 0 0 -> xyz=-0.354 0.128 -0.008 rpy=-1.57 0 0
- joint caster_back_right_joint: origin xyz=-0.177 -0.064 -0.004 rpy=-1.57 0 0 -> xyz=-0.354 -0.128 -0.008 rpy=-1.57 0 0
- joint depth_camera_joint: origin xyz=0.073 0 0.084 rpy=0 0 1.5708 -> xyz=0.146 0 0.168 rpy=0 0.1 1.5708
- joint scan_joint: origin xyz=-0.064 0 0.122 rpy=0 0 0 -> xyz=-0.128 0 0.30 rpy=0 0 0
- joint velodyne_joint: origin xyz=0 0 0.12 rpy=0 0 0 -> xyz=0 0 0.20 rpy=0 0 0
- joint wheel_left_joint: origin xyz=0.0 0.144 0.023 rpy=-1.57 0 0 -> xyz=0.0 0.288 0.046 rpy=-1.57 0 0
- joint wheel_right_joint: origin xyz=0.0 -0.144 0.023 rpy=-1.57 0 0 -> xyz=0.0 -0.288 0.046 rpy=-1.57 0 0
